Commit message: Indent the dimension properties (formatting only)

File: my_arm_description/urdf/dum_e.urdf.xacro (robot description, xacro)
@@ -15,18 +15,18 @@
 <robot name="dum_e" xmlns:xacro="http://www.ros.org/wiki/xacro">
 <!-- ===== Dimensions(m). Change sizes here only. ===== -->
-<xacro:property name="base_plate_length" value="0.05"/>
-<xacro:property name="base_plate_radius" value="0.1"/>
-<xacro:property name="column_length" value="0.3"/>
-<xacro:property name="column_radius" value="0.04"/>
-<xacro:property name="upper_arm_length" value="0.3"/>
-<xacro:property name="upper_arm_radius" value="0.03"/>
-<xacro:property name="forearm_length" value="0.2"/>
-<xacro:property name="forearm_radius" value="0.02"/>
-<xacro:property name="wrist_bracket_size_x" value="0.04"/>
-<xacro:property name="wrist_bracket_size_y" value="0.04"/>
-<xacro:property name="wrist_bracket_length" value="0.06"/>
-<xacro:property name="mount_size_x" value="0.05"/>
-<xacro:property name="mount_size_y" value="0.05"/>
-<xacro:property name="mount_length" value="0.05"/>
+  <xacro:property name="base_plate_length" value="0.05"/>
+  <xacro:property name="base_plate_radius" value="0.1"/>
+  <xacro:property name="column_length" value="0.3"/>
+  <xacro:property name="column_radius" value="0.04"/>
+  <xacro:property name="upper_arm_length" value="0.3"/>
+  <xacro:property name="upper_arm_radius" value="0.03"/>
+  <xacro:property name="forearm_length" value="0.2"/>
+  <xacro:property name="forearm_radius" value="0.02"/>
+  <xacro:property name="wrist_bracket_size_x" value="0.04"/>
+  <xacro:property name="wrist_bracket_size_y" value="0.04"/>
+  <xacro:property name="wrist_bracket_length" value="0.06"/>
+  <xacro:property name="mount_size_x" value="0.05"/>
+  <xacro:property name="mount_size_y" value="0.05"/>
+  <xacro:property name="mount_length" value="0.05"/>
   <!-- ===== Materials ===== -->
   <material name="blue">   <color rgba="0 0 1 1"/>          </material>

Commit message: Compute the column's inertia from its mass and size

File: my_arm_description/urdf/dum_e.urdf.xacro (robot description, xacro)
@@ -19,4 +19,5 @@
   <xacro:property name="column_length" value="0.3"/>
   <xacro:property name="column_radius" value="0.04"/>
+  <xacro:property name="column_mass"   value="0.40"/>   <!-- TODO: real mass -->
   <xacro:property name="upper_arm_length" value="0.3"/>
   <xacro:property name="upper_arm_radius" value="0.03"/>
@@ -70,6 +71,9 @@
     <inertial>
       <origin xyz="0 0 ${column_length / 2}" rpy="0 0 0"/>
-      <mass value="0.40"/>  <!-- TODO: real mass -->
-      <inertia ixx="0.003160" ixy="0" ixz="0" iyy="0.003160" iyz="0" izz="0.000320"/>
+      <mass value="${column_mass}"/>
+      <!-- Solid cylinder about its centre: Ixx = Iyy = m(3r^2 + l^2)/12, Izz = m r^2/2 -->
+      <inertia ixx="${column_mass * (3 * column_radius**2 + column_length**2) / 12}" ixy="0" ixz="0"
+               iyy="${column_mass * (3 * column_radius**2 + column_length**2) / 12}" iyz="0"
+               izz="${column_mass * column_radius**2 / 2}"/>
     </inertial>
   </link>

Commit message: Move the cylinder inertia formula into a macro without changing the robot

File: my_arm_description/urdf/dum_e.urdf.xacro (robot description, xacro)
@@ -30,4 +30,14 @@
   <xacro:property name="mount_size_y" value="0.05"/>
   <xacro:property name="mount_length" value="0.05"/>
+  <xacro:macro name="cylinder_inertial" params="mass radius length">
+  <inertial>
+      <origin xyz="0 0 ${length / 2}" rpy="0 0 0"/>
+      <mass value="${mass}"/>
+      <!-- Solid cylinder about its centre: Ixx = Iyy = m(3r^2 + l^2)/12, Izz = m r^2/2 -->
+      <inertia ixx="${mass * (3 * radius**2 + length**2) / 12}" ixy="0" ixz="0"
+               iyy="${mass * (3 * radius**2 + length**2) / 12}" iyz="0"
+               izz="${mass * radius**2 / 2}"/>
+    </inertial>
+  </xacro:macro>
   <!-- ===== Materials ===== -->
   <material name="blue">   <color rgba="0 0 1 1"/>          </material>
@@ -69,12 +79,5 @@
       <geometry><cylinder length="${column_length}" radius="${column_radius}"/></geometry>
     </collision>
-    <inertial>
-      <origin xyz="0 0 ${column_length / 2}" rpy="0 0 0"/>
-      <mass value="${column_mass}"/>
-      <!-- Solid cylinder about its centre: Ixx = Iyy = m(3r^2 + l^2)/12, Izz = m r^2/2 -->
-      <inertia ixx="${column_mass * (3 * column_radius**2 + column_length**2) / 12}" ixy="0" ixz="0"
-               iyy="${column_mass * (3 * column_radius**2 + column_length**2) / 12}" iyz="0"
-               izz="${column_mass * column_radius**2 / 2}"/>
-    </inertial>
+    <xacro:cylinder_inertial mass="${column_mass}" radius="${column_radius}" length="${column_length}"/>
   </link>
   <!-- ===== J2: shoulder pitch. Positive tips the arm toward +X. ===== -->

Commit message: Use the inertia macro for the upper arm and forearm (now exact values)

File: my_arm_description/urdf/dum_e.urdf.xacro (robot description, xacro)
@@ -22,6 +22,8 @@
   <xacro:property name="upper_arm_length" value="0.3"/>
   <xacro:property name="upper_arm_radius" value="0.03"/>
+  <xacro:property name="upper_arm_mass"   value="0.25"/>   <!-- TODO: real mass -->
   <xacro:property name="forearm_length" value="0.2"/>
   <xacro:property name="forearm_radius" value="0.02"/>
+  <xacro:property name="forearm_mass"   value="0.15"/>   <!-- TODO: real mass -->
   <xacro:property name="wrist_bracket_size_x" value="0.04"/>
   <xacro:property name="wrist_bracket_size_y" value="0.04"/>
@@ -100,9 +102,5 @@
       <geometry><cylinder length="${upper_arm_length}" radius="${upper_arm_radius}"/></geometry>
     </collision>
-    <inertial>
-      <origin xyz="0 0 ${upper_arm_length / 2}" rpy="0 0 0"/>
-      <mass value="0.25"/>  <!-- TODO: real mass -->
-      <inertia ixx="0.001931" ixy="0" ixz="0" iyy="0.001931" iyz="0" izz="0.000112"/>
-    </inertial>
+    <xacro:cylinder_inertial mass="${upper_arm_mass}" radius="${upper_arm_radius}" length="${upper_arm_length}"/>
   </link>
   <!-- ===== J3: elbow pitch ===== -->
@@ -125,9 +123,5 @@
       <geometry><cylinder length="${forearm_length}" radius="${forearm_radius}"/></geometry>
     </collision>
-    <inertial>
-      <origin xyz="0 0 ${forearm_length / 2}" rpy="0 0 0"/>
-      <mass value="0.15"/>  <!-- TODO: real mass -->
-      <inertia ixx="0.000515" ixy="0" ixz="0" iyy="0.000515" iyz="0" izz="0.000030"/>
-    </inertial>
+    <xacro:cylinder_inertial mass="${forearm_mass}" radius="${forearm_radius}" length="${forearm_length}"/>
   </link>
   <!-- ===== J4: wrist pitch (sets the approach angle). Servo: 180 deg range. ===== -->

Commit message: Use the box inertia macro for the wrist bracket and mount (now exact values)

File: my_arm_description/urdf/dum_e.urdf.xacro (robot description, xacro)
@@ -29,7 +29,9 @@
   <xacro:property name="wrist_bracket_size_y" value="0.04"/>
   <xacro:property name="wrist_bracket_length" value="0.06"/>
+  <xacro:property name="wrist_bracket_mass" value="0.06"/>   <!-- TODO: real mass -->
   <xacro:property name="mount_size_x" value="0.05"/>
   <xacro:property name="mount_size_y" value="0.05"/>
   <xacro:property name="mount_length" value="0.05"/>
+  <xacro:property name="mount_mass"         value="0.08"/>   <!-- TODO: real mass -->
   <xacro:macro name="cylinder_inertial" params="mass radius length">
   <inertial>
@@ -40,4 +42,14 @@
                iyy="${mass * (3 * radius**2 + length**2) / 12}" iyz="0"
                izz="${mass * radius**2 / 2}"/>
+    </inertial>
+  </xacro:macro>
+  <xacro:macro name="box_inertial" params="mass x y z">
+  <inertial>
+      <origin xyz="0 0 ${z / 2}" rpy="0 0 0"/>
+      <mass value="${mass}"/>
+      <!-- Solid box about its centre: Ixx = m × (y² + z²) / 12, Iyy = m × (x² + z²) / 12, Izz = m × (x² + y²) / 12 -->
+      <inertia ixx="${mass * (y**2 + z**2) / 12}" ixy="0" ixz="0"
+               iyy="${mass * (x**2 + z**2) / 12}" iyz="0"
+               izz="${mass * (x**2 + y**2) / 12}"/>
     </inertial>
   </xacro:macro>
@@ -144,9 +156,5 @@
       <geometry><box size="${wrist_bracket_size_x} ${wrist_bracket_size_y} ${wrist_bracket_length}"/></geometry>
     </collision>
-    <inertial>
-      <origin xyz="0 0 ${wrist_bracket_length / 2}" rpy="0 0 0"/>
-      <mass value="0.06"/>  <!-- TODO: real mass -->
-      <inertia ixx="0.000026" ixy="0" ixz="0" iyy="0.000026" iyz="0" izz="0.000016"/>
-    </inertial>
+    <xacro:box_inertial mass="${wrist_bracket_mass}" x="${wrist_bracket_size_x}" y="${wrist_bracket_size_y}" z="${wrist_bracket_length}"/>
   </link>
   <!-- ===== J5: wrist roll, about the tool's own axis (local Z). Servo: 180 deg range. ===== -->
@@ -169,9 +177,5 @@
       <geometry><box size="${mount_size_x} ${mount_size_y} ${mount_length}"/></geometry>
     </collision>
-    <inertial>
-      <origin xyz="0 0 ${mount_length / 2}" rpy="0 0 0"/>
-      <mass value="0.08"/>  <!-- TODO: real mass -->
-      <inertia ixx="0.000033" ixy="0" ixz="0" iyy="0.000033" iyz="0" izz="0.000033"/>
-    </inertial>
+    <xacro:box_inertial mass="${mount_mass}" x="${mount_size_x}" y="${mount_size_y}" z="${mount_length}"/>
   </link>
   <!-- ===== tool0: planning tip on the tool-mount face (ADR-005).
